Commit message: Update ra620_1621.urdf

File: 1_1000_hiwin_ra620_1621_support/urdf/ra620_1621.urdf (robot description, URDF)
Before this commit: robot hiwin_ra620_1621, 10 links, 9 joints
Links:
- link base_link: geometry collision mesh filename=package://1_1000_hiwin_ra620_1621_support/meshes/collision/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 scale=0.001 0.001 0.001; visual mesh filename=package://1_1000_hiwin_ra620_1621_support/meshes/visual/bas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 scale=0.001 0.001 0.001
- link link_1: geometry collision mesh filename=package://1_1000_hiwin_ra620_1621_support/meshes/collision/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 scale=0.001 0.001 0.001; visual mesh filename=package://1_1000_hiwin_ra620_1621_support/meshes/visual/lin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 scale=0.001 0.001 0.001
- link link_2: geometry collision mesh filename=package://1_1000_hiwin_ra620_1621_support/meshes/collision/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 scale=0.001 0.001 0.001; visual mesh filename=package://1_1000_hiwin_ra620_1621_support/meshes/visual/lin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 scale=0.001 0.001 0.001
- link link_3: geometry collision mesh filename=package://1_1000_hiwin_ra620_1621_support/meshes/collision/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 scale=0.001 0.001 0.001; visual mesh filename=package://1_1000_hiwin_ra620_1621_support/meshes/visual/lin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 scale=0.001 0.001 0.001
- link link_4: geometry collision mesh filename=package://1_1000_hiwin_ra620_1621_support/meshes/collision/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 scale=0.001 0.001 0.001; visual mesh filename=package://1_1000_hiwin_ra620_1621_support/meshes/visual/lin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 scale=0.001 0.001 0.001
- link link_5: geometry collision mesh filename=package://1_1000_hiwin_ra620_1621_support/meshes/collision/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 scale=0.001 0.001 0.001; visual mesh filename=package://1_1000_hiwin_ra620_1621_support/meshes/visual/lin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 scale=0.001 0.001 0.001
- link link_6: geometry collision mesh filename=package://1_1000_hiwin_ra620_1621_support/meshes/collision/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 scale=0.001 0.001 0.001; visual mesh filename=package://1_1000_hiwin_ra620_1621_support/meshes/visual/lin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 scale=0.001 0.001 0.001
