Commit message: Update ra610_1355_gb.urdf

File: hiwin_ra610_1355_gb_support/urdf/ra610_1355_gb.urdf (robot description, URDF)
Before this commit: robot combine, 7 links, 6 joints
Links:
- link base_link: geometry collision mesh filename=package://hiwin_ra610_1355_gb_support/meshes/ra610_1355/col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 scale=0.001 0.001 0.001; visual mesh filename=package://hiwin_ra610_1355_gb_support/meshes/ra610_1355/vis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 scale=0.001 0.001 0.001
- link link1_v1_1: geometry collision mesh filename=package://hiwin_ra610_1355_gb_support/meshes/ra610_1355/col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 scale=0.001 0.001 0.001; visual mesh filename=package://hiwin_ra610_1355_gb_support/meshes/ra610_1355/vis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 scale=0.001 0.001 0.001
- link link2_v1_1: geometry collision mesh filename=package://hiwin_ra610_1355_gb_support/meshes/ra610_1355/col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 scale=0.001 0.001 0.001; visual mesh filename=package://hiwin_ra610_1355_gb_support/meshes/ra610_1355/vis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 scale=0.001 0.001 0.001
- link link3_v1_1: geometry collision mesh filename=package://hiwin_ra610_1355_gb_support/meshes/ra610_1355/col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 scale=0.001 0.001 0.001; visual mesh filename=package://hiwin_ra610_1355_gb_support/meshes/ra610_1355/vis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 scale=0.001 0.001 0.001
- link link4_v1_1: geometry collision mesh filename=package://hiwin_ra610_1355_gb_support/meshes/ra610_1355/col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 scale=0.001 0.001 0.001; visual mesh filename=package://hiwin_ra610_1355_gb_support/meshes/ra610_1355/vis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 scale=0.001 0.001 0.001
- link link4_v1__1__1: geometry collision mesh filename=package://hiwin_ra610_1355_gb_support/meshes/ra610_1355/col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 scale=0.001 0.001 0.001; visual mesh filename=package://hiwin_ra610_1355_gb_support/meshes/ra610_1355/vis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 scale=0.001 0.001 0.001
- link link5_v1_1: geometry collision mesh filename=package://hiwin_ra610_1355_gb_support/meshes/ra610_1355/col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 scale=0.001 0.001 0.001; visual mesh filename=package://hiwin_ra610_1355_gb_support/meshes/ra610_1355/vis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 scale=0.001 0.001 0.001
