Commit message: Update ra610_1476_gc_macro.xacro

File: hiwin_ra610_1476_gc_support/urdf/ra610_1476_gc_macro.xacro (robot description, xacro)
@@ -7,5 +7,5 @@
             <origin xyz="0 0 0" rpy="0 0 ${pi/2}"/>
             <geometry>
-                <mesh filename="package://hiwin_ra610_1355_gb_support/meshes/visual/base_link.stl" scale="0.001 0.001 0.001"/>
+                <mesh filename="package://hiwin_ra610_1476_gc_support/meshes/visual/base_link.stl" scale="0.001 0.001 0.001"/>
             </geometry>
             <material name="Black">
@@ -16,5 +16,5 @@
             <origin xyz="0 0 0" rpy="0 0 ${pi/2}"/>
             <geometry>
-                <mesh filename="package://hiwin_ra610_1355_gb_support/meshes/collision/base_link.stl" scale="0.001 0.001 0.001"/>
+                <mesh filename="package://hiwin_ra610_1476_gc_support/meshes/collision/base_link.stl" scale="0.001 0.001 0.001"/>
             </geometry>
         </collision>
@@ -24,5 +24,5 @@
             <origin xyz="0 0 0" rpy="0 0 ${pi/2}"/>
             <geometry>
-                <mesh filename="package://hiwin_ra610_1355_gb_support/meshes/visual/link_1.stl" scale="0.001 0.001 0.001"/>
+                <mesh filename="package://hiwin_ra610_1476_gc_support/meshes/visual/link_1.stl" scale="0.001 0.001 0.001"/>
             </geometry>
             <material name="LightGrey">
@@ -33,5 +33,5 @@
             <origin xyz="0 0 0" rpy="0 0 ${pi/2}"/>
             <geometry>
-                <mesh filename="package://hiwin_ra610_1355_gb_support/meshes/collision/link_1.stl" scale="0.001 0.001 0.001"/>
+                <mesh filename="package://hiwin_ra610_1476_gc_support/meshes/collision/link_1.stl" scale="0.001 0.001 0.001"/>
             </geometry>
         </collision>
@@ -41,5 +41,5 @@
             <origin xyz="0 0 0" rpy="0 0 ${pi/2}"/>
             <geometry>
-                <mesh filename="package://hiwin_ra610_1355_gb_support/meshes/visual/link_2.stl" scale="0.001 0.001 0.001"/>
+                <mesh filename="package://hiwin_ra610_1476_gc_support/meshes/visual/link_2.stl" scale="0.001 0.001 0.001"/>
             </geometry>
             <material name="LightGrey">
@@ -50,5 +50,5 @@
             <origin xyz="0 0 0" rpy="0 0 ${pi/2}"/>
             <geometry>
-                <mesh filename="package://hiwin_ra610_1355_gb_support/meshes/collision/link_2.stl" scale="0.001 0.001 0.001"/>
+                <mesh filename="package://hiwin_ra610_1476_gc_support/meshes/collision/link_2.stl" scale="0.001 0.001 0.001"/>
             </geometry>
         </collision>
@@ -58,5 +58,5 @@
             <origin xyz="0 0 0" rpy="0 0 ${pi/2}"/>
             <geometry>
-                <mesh filename="package://hiwin_ra610_1355_gb_support/meshes/visual/link_3.stl" scale="0.001 0.001 0.001"/>
+                <mesh filename="package://hiwin_ra610_1476_gc_support/meshes/visual/link_3.stl" scale="0.001 0.001 0.001"/>
             </geometry>
             <material name="LightGrey">
@@ -67,5 +67,5 @@
             <origin xyz="0 0 0" rpy="0 0 ${pi/2}"/>
             <geometry>
-                <mesh filename="package://hiwin_ra610_1355_gb_support/meshes/collision/link_3.stl" scale="0.001 0.001 0.001"/>
+                <mesh filename="package://hiwin_ra610_1476_gc_support/meshes/collision/link_3.stl" scale="0.001 0.001 0.001"/>
             </geometry>
         </collision>
@@ -75,5 +75,5 @@
             <origin xyz="0 0 0" rpy="0 0 ${pi/2}"/>
             <geometry>
-                <mesh filename="package://hiwin_ra610_1355_gb_support/meshes/visual/link_4.stl" scale="0.001 0.001 0.001"/>
+                <mesh filename="package://hiwin_ra610_1476_gc_support/meshes/visual/link_4.stl" scale="0.001 0.001 0.001"/>
             </geometry>
             <material name="LightGrey">
@@ -84,5 +84,5 @@
             <origin xyz="0 0 0" rpy="0 0 ${pi/2}"/>
             <geometry>
-                <mesh filename="package://hiwin_ra610_1355_gb_support/meshes/collision/link_4.stl" scale="0.001 0.001 0.001"/>
+                <mesh filename="package://hiwin_ra610_1476_gc_support/meshes/collision/link_4.stl" scale="0.001 0.001 0.001"/>
             </geometry>
         </collision>
@@ -92,5 +92,5 @@
             <origin xyz="0 0 0" rpy="0 0 ${pi/2}"/>
             <geometry>
-                <mesh filename="package://hiwin_ra610_1355_gb_support/meshes/visual/link_5.stl" scale="0.001 0.001 0.001"/>
+                <mesh filename="package://hiwin_ra610_1476_gc_support/meshes/visual/link_5.stl" scale="0.001 0.001 0.001"/>
             </geometry>
             <material name="LightGrey">
@@ -101,5 +101,5 @@
             <origin xyz="0 0 0" rpy="0 0 ${pi/2}"/>
             <geometry>
-                <mesh filename="package://hiwin_ra610_1355_gb_support/meshes/collision/link_5.stl" scale="0.001 0.001 0.001"/>
+                <mesh filename="package://hiwin_ra610_1476_gc_support/meshes/collision/link_5.stl" scale="0.001 0.001 0.001"/>
             </geometry>
         </collision>
@@ -109,5 +109,5 @@
             <origin xyz="0 0 0" rpy="0 0 ${pi/2}"/>
             <geometry>
-                <mesh filename="package://hiwin_ra610_1355_gb_support/meshes/visual/link_6.stl" scale="0.001 0.001 0.001"/>
+                <mesh filename="package://hiwin_ra610_1476_gc_support/meshes/visual/link_6.stl" scale="0.001 0.001 0.001"/>
             </geometry>
             <material name="LightGrey">
@@ -118,5 +118,5 @@
             <origin xyz="0 0 0" rpy="0 0 ${pi/2}"/>
             <geometry>
-                <mesh filename="package://hiwin_ra610_1355_gb_support/meshes/collision/link_6.stl" scale="0.001 0.001 0.001"/>
+                <mesh filename="package://hiwin_ra610_1476_gc_support/meshes/collision/link_6.stl" scale="0.001 0.001 0.001"/>
             </geometry>
         </collision>

Commit message: Update ra610_1476_gc_macro.xacro

File: hiwin_ra610_1476_gc_support/urdf/ra610_1476_gc_macro.xacro (robot description, xacro)
@@ -39,5 +39,5 @@
     <link name="${prefix}link_2" >
         <visual>
-            <origin xyz="0 0 0" rpy="0 0 ${pi/2}"/>
+            <origin xyz="-0.106 -0.14 -0.257" rpy="0 0 ${pi/2}"/>
             <geometry>
                 <mesh filename="package://hiwin_ra610_1476_gc_support/meshes/visual/link_2.stl" scale="0.001 0.001 0.001"/>
@@ -48,5 +48,5 @@
         </visual>
         <collision>
-            <origin xyz="0 0 0" rpy="0 0 ${pi/2}"/>
+            <origin xyz="-0.106 -0.14 -0.257" rpy="0 0 ${pi/2}"/>
             <geometry>
                 <mesh filename="package://hiwin_ra610_1476_gc_support/meshes/collision/link_2.stl" scale="0.001 0.001 0.001"/>
@@ -56,5 +56,5 @@
     <link name="${prefix}link_3" >
         <visual>
-            <origin xyz="0 0 0" rpy="0 0 ${pi/2}"/>
+            <origin xyz="-0.136 -0.14 -0.897" rpy="0 0 ${pi/2}"/>
             <geometry>
                 <mesh filename="package://hiwin_ra610_1476_gc_support/meshes/visual/link_3.stl" scale="0.001 0.001 0.001"/>
@@ -65,5 +65,5 @@
         </visual>
         <collision>
-            <origin xyz="0 0 0" rpy="0 0 ${pi/2}"/>
+            <origin xyz="-0.136 -0.14 -0.897" rpy="0 0 ${pi/2}"/>
             <geometry>
                 <mesh filename="package://hiwin_ra610_1476_gc_support/meshes/collision/link_3.stl" scale="0.001 0.001 0.001"/>
@@ -73,5 +73,5 @@
     <link name="${prefix}link_4" >
         <visual>
-            <origin xyz="0 0 0" rpy="0 0 ${pi/2}"/>
+            <origin xyz="0.0 -0.2895 -1.057" rpy="0 0 0"/>
             <geometry>
                 <mesh filename="package://hiwin_ra610_1476_gc_support/meshes/visual/link_4.stl" scale="0.001 0.001 0.001"/>
@@ -82,5 +82,5 @@
         </visual>
         <collision>
-            <origin xyz="0 0 0" rpy="0 0 ${pi/2}"/>
+            <origin xyz="0.0 -0.2895 -1.057" rpy="0 0 0"/>
             <geometry>
                 <mesh filename="package://hiwin_ra610_1476_gc_support/meshes/collision/link_4.stl" scale="0.001 0.001 0.001"/>
@@ -90,5 +90,5 @@
     <link name="${prefix}link_5" >
         <visual>
-            <origin xyz="0 0 0" rpy="0 0 ${pi/2}"/>
+            <origin xyz="0.001 -0.8065 -1.057" rpy="0 0 ${pi/2}"/>
             <geometry>
                 <mesh filename="package://hiwin_ra610_1476_gc_support/meshes/visual/link_5.stl" scale="0.001 0.001 0.001"/>
@@ -99,5 +99,5 @@
         </visual>
         <collision>
-            <origin xyz="0 0 0" rpy="0 0 ${pi/2}"/>
+            <origin xyz="0.001 -0.8065 -1.057" rpy="0 0 ${pi/2}"/>
             <geometry>
                 <mesh filename="package://hiwin_ra610_1476_gc_support/meshes/collision/link_5.stl" scale="0.001 0.001 0.001"/>
@@ -107,5 +107,5 @@
     <link name="${prefix}link_6" >
         <visual>
-            <origin xyz="0 0 0" rpy="0 0 ${pi/2}"/>
+            <origin xyz="0.002 -0.8065 -0.974" rpy="0 0 ${pi/2}"/>
             <geometry>
                 <mesh filename="package://hiwin_ra610_1476_gc_support/meshes/visual/link_6.stl" scale="0.001 0.001 0.001"/>
@@ -116,5 +116,5 @@
         </visual>
         <collision>
-            <origin xyz="0 0 0" rpy="0 0 ${pi/2}"/>
+            <origin xyz="0.002 -0.8065 -0.974" rpy="0 0 ${pi/2}"/>
             <geometry>
                 <mesh filename="package://hiwin_ra610_1476_gc_support/meshes/collision/link_6.stl" scale="0.001 0.001 0.001"/>
@@ -124,43 +124,43 @@
     <!-- joints: main serial chain -->
     <joint name="${prefix}joint_1" type="revolute">
-        <origin xyz="0.0 0.0 0.191" rpy="0.0 0.0 0.0" />
+        <origin xyz="0.0 0.0 0.0" rpy="0.0 0.0 0.0" />
         <parent link="${prefix}base_link" />
         <child link="${prefix}link_1" />
-        <axis xyz="0 0 1" />
+        <axis xyz="0.0 0.0 1.0" />
         <limit lower="-2.8792" upper="2.8792" effort="0" velocity="2.618"/>
     </joint>
     <joint name="${prefix}joint_2" type="revolute">
-        <origin xyz="0.0 0.140 0.255" rpy="0.0 0.0 0.0" />
+        <origin xyz="0.106 0.14 0.257" rpy="0.0 0.0 0.0" />
         <parent link="${prefix}link_1" />
         <child link="${prefix}link_2" />
-        <axis xyz="1 0 0" />
+        <axis xyz="1.0 0.0 0.0" />
         <limit lower="-2.1812" upper="1.4832" effort="0" velocity="2.618"/>
     </joint>
     <joint name="${prefix}joint_3" type="revolute">
-        <origin xyz="0.0 0.000 0.642" rpy="0.0 0.0 0.0" />
+        <origin xyz="0.03 0.0 0.64" rpy="0.0 0.0 0.0" />
         <parent link="${prefix}link_2" />
         <child link="${prefix}link_3" />
-        <axis xyz="1 0 0" />
+        <axis xyz="-1.0 0.0 0.0" />
         <limit lower="-0.9597" upper="3.2282" effort="0" velocity="2.618"/>
     </joint>
     <joint name="${prefix}joint_4" type="revolute">
-        <origin xyz="0.0 0.1495 0.160" rpy="0.0 0.0 0.0" />
+        <origin xyz="-0.136 0.1495 0.16" rpy="0.0 0.0 0.0" />
         <parent link="${prefix}link_3" />
         <child link="${prefix}link_4" />
-        <axis xyz="0 1 0" />
+        <axis xyz="0.0 1.0 0.0" />
         <limit lower="-3.3155" upper="3.3155" effort="0" velocity="2.618"/>
     </joint>
     <joint name="${prefix}joint_5" type="revolute">
-        <origin xyz="0.0 0.4025 0.000" rpy="0.0 0.0 0.0" />
+        <origin xyz="-0.001 0.517 0.0" rpy="0.0 0.0 0.0" />
         <parent link="${prefix}link_4" />
         <child link="${prefix}link_5" />
-        <axis xyz="1 0 0" />
+        <axis xyz="1.0 -0.0 -0.0" />
         <limit lower="-2.0067" upper="2.0067" effort="0" velocity="2.618"/>
     </joint>
     <joint name="${prefix}joint_6" type="revolute">
-        <origin xyz="0.0 0.080 0.0" rpy="0.0 0.0 0.0" />
+        <origin xyz="-0.001 0.0 -0.083" rpy="0.0 0.0 0.0" />
         <parent link="${prefix}link_5" />
         <child link="${prefix}link_6" />
-        <axis xyz="0 1 0" />
+        <axis xyz="0.0 0.0 -1.0" />
         <limit lower="-3.1415" upper="3.1415" effort="0" velocity="2.618"/>
     </joint>
