Commit message: Update ra610_1476_gc.urdf

File: hiwin_ra610_1476_gc_support/urdf/ra610_1476_gc.urdf (robot description, URDF)
Before this commit: robot ra610_1476_gc, 7 links, 6 joints
Joints:
- joint Revolute 1: origin xyz=0.0 0.0 0.0 rpy=0 0 0 -> xyz=0.0 0.0 0.191 rpy=0 0 0
- joint Revolute 2: origin xyz=0.106 0.14 0.257 rpy=0 0 0 -> xyz=0.0 0.140 0.255 rpy=0 0 0
- joint Revolute 3: origin xyz=0.03 0.0 0.64 rpy=0 0 0 -> xyz=0.0 0.000 0.642 rpy=0 0 0
- joint Revolute 4: origin xyz=-0.136 0.1495 0.16 rpy=0 0 0 -> xyz=0.0 0.1495 0.160 rpy=0 0 0
- joint Revolute 5: origin xyz=-0.001 0.517 0.0 rpy=0 0 0 -> xyz=0.0 0.4025 0.000 rpy=0 0 0
- joint Revolute 6: origin xyz=-0.001 0.0 -0.083 rpy=0 0 0 -> xyz=0.0 0.080 0.0 rpy=0 0 0

Commit message: Update ra610_1476_gc.urdf

File: hiwin_ra610_1476_gc_support/urdf/ra610_1476_gc.urdf (robot description, URDF)
Before this commit: robot ra610_1476_gc, 7 links, 6 joints
Links:
- removed link link5_v1_1
- added link base
- added link flange
- added link link_6; collision mesh filename=package://hiwin_ra610_1476_support/meshes/ra610_1476/collis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 scale=0.001 0.001 0.001; visual mesh filename=package://hiwin_ra610_1476_support/meshes/ra610_1476/visual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 scale=0.001 0.001 0.001
- added link tool0
- link base_link: mass 12.14290466451666 -> None; geometry collision mesh filename=package://hiwin_ra610_1476_support/meshes/ra610_1476/collis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 scale=0.001 0.001 0.001; visual mesh filename=package://hiwin_ra610_1476_support/meshes/ra610_1476/visual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 scale=0.001 0.001 0.001
- link link_1: mass 20.145436969150147 -> None; geometry collision mesh filename=package://hiwin_ra610_1476_support/meshes/ra610_1476/collis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 scale=0.001 0.001 0.001; visual mesh filename=package://hiwin_ra610_1476_support/meshes/ra610_1476/visual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 scale=0.001 0.001 0.001
- link link_2: mass 7.125940242438544 -> None; geometry collision mesh filename=package://hiwin_ra610_1476_support/meshes/ra610_1476/collis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 scale=0.001 0.001 0.001; visual mesh filename=package://hiwin_ra610_1476_support/meshes/ra610_1476/visual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 scale=0.001 0.001 0.001
- link link_3: mass 8.570278236005578 -> None; geometry collision mesh filename=package://hiwin_ra610_1476_support/meshes/ra610_1476/collis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 scale=0.001 0.001 0.001; visual mesh filename=package://hiwin_ra610_1476_support/meshes/ra610_1476/visual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 scale=0.001 0.001 0.001
- link link_4: mass 6.4431594647450385 -> None; geometry collision mesh filename=package://hiwin_ra610_1476_support/meshes/ra610_1476/collis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 scale=0.001 0.001 0.001; visual mesh filename=package://hiwin_ra610_1476_support/meshes/ra610_1476/visual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 scale=0.001 0.001 0.001
- link link_5: mass 0.9514751636393539 -> None; geometry collision mesh filename=package://hiwin_ra610_1476_support/meshes/ra610_1476/collis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 scale=0.001 0.001 0.001; visual mesh filename=package://hiwin_ra610_1476_support/meshes/ra610_1476/visual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 scale=0.001 0.001 0.001
Joints:
- removed joint Revolute 1
- removed joint Revolute 2
- removed joint Revolute 3
- removed joint Revolute 4
- removed joint Revolute 5
- removed joint Revolute 6
- added joint base_link-base: type fixed, parent base_link, child base, origin xyz=0.000076 0.003189 0.375960 rpy=0 0 0
- added joint joint_1: type revolute, parent base_link, child link_1, origin xyz=0.0 0.0 0.191 rpy=0.0 0.0 0.0, axis 0 0 1, limit lower=-2.8792 upper=2.8792 effort=0 velocity=2.618
- added joint joint_2: type revolute, parent link_1, child link_2, origin xyz=0.0 0.140 0.255 rpy=0.0 0.0 0.0, axis 1 0 0, limit lower=-2.1812 upper=1.4832 effort=0 velocity=2.618
- added joint joint_3: type revolute, parent link_2, child link_3, origin xyz=0.0 0.000 0.642 rpy=0.0 0.0 0.0, axis 1 0 0, limit lower=-0.9597 upper=3.2282 effort=0 velocity=2.618
- added joint joint_4: type revolute, parent link_3, child link_4, origin xyz=0.0 0.1495 0.160 rpy=0.0 0.0 0.0, axis 0 1 0, limit lower=-3.3155 upper=3.3155 effort=0 velocity=2.618
- added joint joint_5: type revolute, parent link_4, child link_5, origin xyz=0.0 0.4025 0.000 rpy=0.0 0.0 0.0, axis 1 0 0, limit lower=-2.0067 upper=2.0067 effort=0 velocity=2.618
- added joint joint_6: type revolute, parent link_5, child link_6, origin xyz=0.0 0.080 0.0 rpy=0.0 0.0 0.0, axis 0 1 0, limit lower=-3.1415 upper=3.1415 effort=0 velocity=2.618
- added joint joint_6-flange: type fixed, parent link_6, child flange, origin xyz=0 0.016 0 rpy=0 0 0
- added joint link_6-tool0: type fixed, parent link_6, child tool0, origin xyz=0 0.020 0.0 rpy=0.0 ${-pi/2.0} ${-pi/2.0}

Commit message: Update ra610_1476_gc.urdf

File: hiwin_ra610_1476_gc_support/urdf/ra610_1476_gc.urdf (robot description, URDF)
Before this commit: robot hiwin_ra610_1476, 10 links, 9 joints
Joints:
- joint link_6-tool0: origin xyz=0 0.020 0.0 rpy=0.0 ${-pi/2.0} ${-pi/2.0} -> xyz=0 0.020 0.0 rpy=0.0 -1.57079632679 -1.57079632679

Commit message: Update ra610_1476_gc.urdf

File: hiwin_ra610_1476_gc_support/urdf/ra610_1476_gc.urdf (robot description, URDF)
Before this commit: robot hiwin_ra610_1476, 10 links, 9 joints
Links:
- link base_link: geometry collision mesh filename=package://hiwin_ra610_1476_gc_support/meshes/ra610_1476/col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 scale=0.001 0.001 0.001; visual mesh filename=package://hiwin_ra610_1476_gc_support/meshes/ra610_1476/vis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 scale=0.001 0.001 0.001
- link link_1: geometry collision mesh filename=package://hiwin_ra610_1476_gc_support/meshes/ra610_1476/col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 scale=0.001 0.001 0.001; visual mesh filename=package://hiwin_ra610_1476_gc_support/meshes/ra610_1476/vis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 scale=0.001 0.001 0.001
- link link_2: geometry collision mesh filename=package://hiwin_ra610_1476_gc_support/meshes/ra610_1476/col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 scale=0.001 0.001 0.001; visual mesh filename=package://hiwin_ra610_1476_gc_support/meshes/ra610_1476/vis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 scale=0.001 0.001 0.001
- link link_3: geometry collision mesh filename=package://hiwin_ra610_1476_gc_support/meshes/ra610_1476/col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 scale=0.001 0.001 0.001; visual mesh filename=package://hiwin_ra610_1476_gc_support/meshes/ra610_1476/vis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 scale=0.001 0.001 0.001
- link link_4: geometry collision mesh filename=package://hiwin_ra610_1476_gc_support/meshes/ra610_1476/col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 scale=0.001 0.001 0.001; visual mesh filename=package://hiwin_ra610_1476_gc_support/meshes/ra610_1476/vis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 scale=0.001 0.001 0.001
- link link_5: geometry collision mesh filename=package://hiwin_ra610_1476_gc_support/meshes/ra610_1476/col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 scale=0.001 0.001 0.001; visual mesh filename=package://hiwin_ra610_1476_gc_support/meshes/ra610_1476/vis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 scale=0.001 0.001 0.001
- link link_6: geometry collision mesh filename=package://hiwin_ra610_1476_gc_support/meshes/ra610_1476/col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 scale=0.001 0.001 0.001; visual mesh filename=package://hiwin_ra610_1476_gc_support/meshes/ra610_1476/vis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 scale=0.001 0.001 0.001

Commit message: Update ra610_1476_gc.urdf

File: hiwin_ra610_1476_gc_support/urdf/ra610_1476_gc.urdf (robot description, URDF)
Before this commit: robot hiwin_ra610_1476, 10 links, 9 joints
Links:
- link base_link: geometry collision mesh filename=package://hiwin_ra610_1476_gc_support/meshes/ra610_1476/col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; visual mesh filename=package://hiwin_ra610_1476_gc_support/meshes/ra610_1476/vis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
- link link_1: geometry collision mesh filename=package://hiwin_ra610_1476_gc_support/meshes/ra610_1476/col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; visual mesh filename=package://hiwin_ra610_1476_gc_support/meshes/ra610_1476/vis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
- link link_2: geometry collision mesh filename=package://hiwin_ra610_1476_gc_support/meshes/ra610_1476/col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; visual mesh filename=package://hiwin_ra610_1476_gc_support/meshes/ra610_1476/vis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
- link link_3: geometry collision mesh filename=package://hiwin_ra610_1476_gc_support/meshes/ra610_1476/col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; visual mesh filename=package://hiwin_ra610_1476_gc_support/meshes/ra610_1476/vis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
- link link_4: geometry collision mesh filename=package://hiwin_ra610_1476_gc_support/meshes/ra610_1476/col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; visual mesh filename=package://hiwin_ra610_1476_gc_support/meshes/ra610_1476/vis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
- link link_5: geometry collision mesh filename=package://hiwin_ra610_1476_gc_support/meshes/ra610_1476/col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; visual mesh filename=package://hiwin_ra610_1476_gc_support/meshes/ra610_1476/vis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
- link link_6: geometry collision mesh filename=package://hiwin_ra610_1476_gc_support/meshes/ra610_1476/col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; visual mesh filename=package://hiwin_ra610_1476_gc_support/meshes/ra610_1476/vis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

Commit message: Update ra610_1476_gc.urdf

File: hiwin_ra610_1476_gc_support/urdf/ra610_1476_gc.urdf (robot description, URDF)
Before this commit: robot hiwin_ra610_1476, 10 links, 9 joints
Joints:
- joint joint_2: origin xyz=0.0 0.140 0.255 rpy=0.0 0.0 0.0 -> xyz=0.0 0.0 0.0 rpy=0.0 0.0 0.0
- joint joint_3: origin xyz=0.0 0.000 0.642 rpy=0.0 0.0 0.0 -> xyz=0.0 0.0 0.0 rpy=0.0 0.0 0.0
- joint joint_4: origin xyz=0.0 0.1495 0.160 rpy=0.0 0.0 0.0 -> xyz=0.0 0.0 0.0 rpy=0.0 0.0 0.0
- joint joint_5: origin xyz=0.0 0.4025 0.000 rpy=0.0 0.0 0.0 -> xyz=0.0 0.0 0.0 rpy=0.0 0.0 0.0
- joint joint_6: origin xyz=0.0 0.080 0.0 rpy=0.0 0.0 0.0 -> xyz=0.0 0.0 0.0 rpy=0.0 0.0 0.0
