Commit message: Add files via upload

File: hiwin_ra610_1476_support/urdf/ra610_1476.urdf (robot description, URDF)
Before this commit: robot None, 0 links, 0 joints
Links:
- added link base
- added link base_link; collision mesh filename=package://hiwin_ra610_1476_support/meshes/collision/base_li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 scale=0.001 0.001 0.001; visual mesh filename=package://hiwin_ra610_1476_support/meshes/visual/base_link.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 scale=0.001 0.001 0.001
- added link flange
- added link link_1; collision mesh filename=package://hiwin_ra610_1476_support/meshes/collision/link_1.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 scale=0.001 0.001 0.001; visual mesh filename=package://hiwin_ra610_1476_support/meshes/visual/link_1.stl scale=0.001 0.001 0.001
- added link link_2; collision mesh filename=package://hiwin_ra610_1476_support/meshes/collision/link_2.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 scale=0.001 0.001 0.001; visual mesh filename=package://hiwin_ra610_1476_support/meshes/visual/link_2.stl scale=0.001 0.001 0.001
- added link link_3; collision mesh filename=package://hiwin_ra610_1476_support/meshes/collision/link_3.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 scale=0.001 0.001 0.001; visual mesh filename=package://hiwin_ra610_1476_support/meshes/visual/link_3.stl scale=0.001 0.001 0.001
- added link link_4; collision mesh filename=package://hiwin_ra610_1476_support/meshes/collision/link_4.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 scale=0.001 0.001 0.001; visual mesh filename=package://hiwin_ra610_1476_support/meshes/visual/link_4.stl scale=0.001 0.001 0.001
- added link link_5; collision mesh filename=package://hiwin_ra610_1476_support/meshes/collision/link_5.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 scale=0.001 0.001 0.001; visual mesh filename=package://hiwin_ra610_1476_support/meshes/visual/link_5.stl scale=0.001 0.001 0.001
- added link link_6; collision mesh filename=package://hiwin_ra610_1476_support/meshes/collision/link_6.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 scale=0.001 0.001 0.001; visual mesh filename=package://hiwin_ra610_1476_support/meshes/visual/link_6.stl scale=0.001 0.001 0.001
- added link tool0
Joints:
- added joint base_link-base: type fixed, parent base_link, child base, origin xyz=0.000076 0.003189 0.375960 rpy=0 0 0
- added joint joint_1: type revolute, parent base_link, child link_1, origin xyz=0.0 0.0 0.2085 rpy=0.0 0.0 0.0, axis 0 0 1, limit lower=-2.8792 upper=2.8792 effort=0 velocity=2.618
- added joint joint_2: type revolute, parent link_1, child link_2, origin xyz=0.000 0.140 0.240 rpy=0.0 0.0 0.0, axis 1 0 0, limit lower=-2.1812 upper=1.4832 effort=0 velocity=2.618
- added joint joint_3: type revolute, parent link_2, child link_3, origin xyz=0.0 0.0 0.64 rpy=0.0 0.0 0.0, axis 1 0 0, limit lower=-0.9597 upper=3.2282 effort=0 velocity=2.618
- added joint joint_4: type revolute, parent link_3, child link_4, origin xyz=0.0 0.1495 0.16 rpy=0.0 0.0 0.0, axis 0 1 0, limit lower=-3.3155 upper=3.3155 effort=0 velocity=2.618
- added joint joint_5: type revolute, parent link_4, child link_5, origin xyz=0.0 0.5285 0.0 rpy=0.0 0.0 0.0, axis 1 0 0, limit lower=-2.0067 upper=2.0067 effort=0 velocity=2.618
- added joint joint_6: type revolute, parent link_5, child link_6, origin xyz=0.0 0.0 0.0 rpy=0.0 0.0 0.0, axis 0 1 0, limit lower=-3.1415 upper=3.1415 effort=0 velocity=2.618
- added joint joint_6-flange: type fixed, parent link_6, child flange, origin xyz=0 0.016 0 rpy=0 0 0
- added joint link_6-tool0: type fixed, parent link_6, child tool0, origin xyz=0 0.020 0.0 rpy=0.0 -1.5707963267948966 -1.5707963267948966
